File: MCU-2627.kicad_sch (KiCad schematic)
At the start: 0 parts

Commit message: MCU + decoup caps added
Added MCU and decoup caps to schematic
Parts:
- added C1, C10, C2, C3, C4, C5, C6, C7, C8, C9: 100n, symbol Device:C_Small
- added U1: RP2350B, Package_DFN_QFN:QFN-80-1EP_10x10mm_P0.4mm_EP3.4x3.4mm, symbol MCU_RaspberryPi:RP2350B
Connections:
- new net: U1.10 (DVDD), U1.32 (DVDD), U1.51 (DVDD)
- new net: U1.15 (IOVDD), U1.24 (IOVDD), U1.29 (IOVDD), U1.41 (IOVDD), U1.5 (IOVDD), U1.50 (IOVDD), U1.60 (IOVDD), U1.76 (IOVDD)
- new net +1V1: C10.1, C8.1, C9.1
- new net +3V3: C1.1, C2.1, C3.1, C4.1, C5.1, C6.1, C7.1
- new net GND: C1.2, C10.2, C2.2, C3.2, C4.2, C5.2, C6.2, C7.2, C8.2, C9.2

Commit message: Added gnd, 3.3V, and 5V connections to mcu
Connections:
- net +1V1: now also U1.10 (DVDD), U1.32 (DVDD), U1.51 (DVDD)
- net +3V3: now also U1.15 (IOVDD), U1.24 (IOVDD), U1.29 (IOVDD), U1.41 (IOVDD), U1.5 (IOVDD), U1.50 (IOVDD), U1.60 (IOVDD), U1.76 (IOVDD)
- net GND: now also U1.81 (GND)
Changed lines of the file:
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@@
+	)
+	(symbol
+		(lib_id "power:+3V3")
+		(at 119.38 54.61 0)
+		(unit 1)
+		(body_style 1)
+		(exclude_from_sim no)
+		(in_bom yes)
+		(on_board yes)
+		(in_pos_files yes)
+		(dnp no)
+		(fields_autoplaced yes)
+		(property "Reference" "#PWR06"
+			(at 119.38 58.42 0)
+			(hide yes)
+			(show_name no)
+			(do_not_autoplace no)
+			(effects
+				(font
+					(size 1.27 1.27)
+				)
+			)
+		)
+		(property "Value" "+3V3"
+			(at 119.38 49.53 0)
+			(show_name no)
+			(do_not_autoplace no)
+			(effects
+				(font
+					(size 1.27 1.27)
+				)
+			)
+		)
+		(property "Footprint" ""
+			(at 119.38 54.61 0)
+			(hide yes)
+			(show_name no)
+			(do_not_autoplace no)
+			(effects
+				(font
+					(size 1.27 1.27)
+				)
+			)
+		)
+		(property "Datasheet" ""
+			(at 119.38 54.61 0)
+			(hide yes)
+			(show_name no)
+			(do_not_autoplace no)
+			(effects
+				(font
+					(size 1.27 1.27)
+				)
+			)
+		)
+		(property "Description" "Power symbol creates a global label with name \"+3V3\""
+			(at 119.38 54.61 0)
+			(hide yes)
+			(show_name no)
+			(do_not_autoplace no)
+			(effects
+				(font
+					(size 1.27 1.27)
+				)
+			)
+		)
+		(pin "1"
+		)
+		(instances
+			(project "MCU-2627"
+				(path "/d48ada1f-57f1-40f0-bdfe-1ee42f4b28b2"
+					(reference "#PWR06")
+					(unit 1)
+				)
+			)
+		)
 	)
 	(symbol
@@
 					(unit 1)
 				)
+			)
+		)
+	)
+	(symbol
+		(lib_id "power:GND")
+		(at 121.92 168.91 0)
+		(unit 1)
+		(body_style 1)
+		(exclude_from_sim no)
+		(in_bom yes)
+		(on_board yes)
+		(in_pos_files yes)
+		(dnp no)
+		(fields_autoplaced yes)
+		(property "Reference" "#PWR07"
+			(at 121.92 175.26 0)
+			(hide yes)
+			(show_name no)
+			(do_not_autoplace no)
+			(effects
+				(font
+					(size 1.27 1.27)
+				)
+			)
+		)
+		(property "Value" "GND"
+			(at 121.92 173.99 0)
+			(show_name no)
+			(do_not_autoplace no)
+			(effects
+				(font
+					(size 1.27 1.27)
+				)
+			)
+		)
+		(property "Footprint" ""
+			(at 121.92 168.91 0)
+			(hide yes)
+			(show_name no)
+			(do_not_autoplace no)
+			(effects
+				(font
+					(size 1.27 1.27)
+				)
+			)
+		)
+		(property "Datasheet" ""
+			(at 121.92 168.91 0)
+			(hide yes)
+			(show_name no)
+			(do_not_autoplace no)
+			(effects
+				(font
+					(size 1.27 1.27)
+				)
+			)
+		)
+		(property "Description" "Power symbol creates a global label with name \"GND\" , ground"
+			(at 121.92 168.91 0)
+			(hide yes)
+			(show_name no)
+			(do_not_autoplace no)
+			(effects
+				(font
+					(size 1.27 1.27)
+				)
+			)
+		)
+		(pin "1"
+		)
+		(instances
+			(project "MCU-2627"
+				(path "/d48ada1f-57f1-40f0-bdfe-1ee42f4b28b2"
+					(reference "#PWR07")
+					(unit 1)
+				)
+			)
+		)
+	)
+	(symbol
+		(lib_id "power:+1V1")
+		(at 134.62 54.61 0)
+		(unit 1)
+		(body_style 1)
+		(exclude_from_sim no)
+		(in_bom yes)
+		(on_board yes)
+		(in_pos_files yes)
+		(dnp no)
+		(fields_autoplaced yes)
+		(property "Reference" "#PWR05"
+			(at 134.62 58.42 0)
+			(hide yes)
+			(show_name no)
+			(do_not_autoplace no)
+			(effects
+				(font
+					(size 1.27 1.27)
+				)
+			)
+		)
+		(property "Value" "+1V1"
+			(at 134.62 49.53 0)
+			(show_name no)
+			(do_not_autoplace no)
+			(effects
+				(font
+					(size 1.27 1.27)
+				)
+			)
+		)
+		(property "Footprint" ""
+			(at 134.62 54.61 0)
+			(hide yes)
+			(show_name no)
+			(do_not_autoplace no)
+			(effects
+				(font
+					(size 1.27 1.27)
+				)
+			)
+		)
+		(property "Datasheet" ""
+			(at 134.62 54.61 0)
+			(hide yes)
+			(show_name no)
+			(do_not_autoplace no)
+			(effects
+				(font
+					(size 1.27 1.27)
+				)
+			)
+		)
+		(property "Description" "Power symbol creates a global label with name \"+1V1\""
+			(at 134.62 54.61 0)
+			(hide yes)
+			(show_name no)
+			(do_not_autoplace no)
+			(effects
+				(font
+					(size 1.27 1.27)
+				)
+			)
+		)
+		(pin "1"
+		)
+		(instances
+			(project "MCU-2627"
+				(path "/d48ada1f-57f1-40f0-bdfe-1ee42f4b28b2"
+					(reference "#PWR05")
+					(unit 1)
+				)

Commit message: added usb, debug connector, and internal regulator circuitry
Parts:
- added C11, C12, C13: 4.7u, symbol Device:C_Small
- added C14, C15: 15p, symbol Device:C_Small
- added C16, C17: 10u, symbol Device:C_Small
- added C18: 100n, symbol Device:C_Small
- added J1: SM03B-SRSS-TBLFSN, CONN_SM03B-SRSS-TB_JST, symbol Symbols:SM03B-SRSS-TBLFSN
- added J2: USB_C_Receptacle_USB2.0_14P, symbol Connector:USB_C_Receptacle_USB2.0_14P
- added J3: Conn_01x13_Pin, symbol Connector:Conn_01x13_Pin
- added J4: Conn_2Rows-51Pins, symbol Connector_Generic:Conn_2Rows-51Pins
- added L1: 3.3u, symbol Device:L
- added R1: R, symbol Device:R
- added R2: 1k, symbol Device:R
- added R3, R4: 27, symbol Device:R
- added R5, R6: 5.1k, symbol Device:R
- added U2: W25Q128JVSIQ, SOIC_128JVSIQ_WIN, symbol Symbols:W25Q128JVSIQ
- added U3: NCP1117ST33T3G, SOT223-3_ONS, symbol Symbols:NCP1117ST33T3G
- added X1: ABM8-272-T3, ABM8-272-T3_ABR, symbol 2026-10-15_16-24-31:ABM8-272-T3
Connections:
- net +1V1: now also U1.65 (VREG_FB), C13.2, L1.1
- net +3V3: now also U1.59 (ADC_AVDD), U1.64 (VREG_VIN), U1.68 (USB_OTP_VDD), U1.69 (QSPI_IOVDD), C12.2, C16.1, C18.1, R1.1, U2.8 (VCC), U3.2 (OUTPUT)
- net GND: now also U1.62 (VREG_PGND), C11.2, C12.1, C13.1, C14.2, C15.2, C16.2, C17.2, C18.2, J1.2, J2.A1 (GND), J2.A12 (GND), J2.B1 (GND), J2.B12 (GND), J2.SH (SHIELD), R5.2, R6.2, U2.4 (GND), U3.1 (ADJUST/GROUND), X1.2, X1.4
- net at U1.30 (XIN): now also C15.1, X1.1
- net at U1.31 (XOUT): now also R2.2
- net at U1.33 (SWCLK): now also J1.1
- net at U1.34 (SWDIO): now also J1.3
- net at U1.61 (VREG_AVDD): now also C11.1, R1.2
- net at U1.63 (VREG_LX): now also L1.2
- net at U1.66 (USB_DM): now also R3.2
- net at U1.67 (USB_DP): now also R4.2
- net QSPI_SD3: now reaches U1.70 (QSPI_SD3)
- net QSPI_SD3: now also U2.7 (/HOLD_or_/RESET_(IO3))
- net QSPI_SCLK: now reaches U1.71 (QSPI_SCLK)
- net QSPI_SCLK: now also U2.6 (CLK)
- net QSPI_SD0: now reaches U1.72 (QSPI_SD0)
- net QSPI_SD0: now also U2.5 (DI_(IO0))
- net QSPI_SD2: now reaches U1.73 (QSPI_SD2)
- net QSPI_SD2: now also U2.3
- net QSPI_SD1: now reaches U1.74 (QSPI_SD1)
- net QSPI_SD1: now also U2.2 (DO_(IO1))
- net QSPI_SS: now reaches U1.75 (~{QSPI_SS})
- net QSPI_SS: now also U2.1 (/CS)
- new net: C14.1, R2.1, X1.3
- new net: C17.1, J2.A4 (VBUS), J2.A9 (VBUS), J2.B4 (VBUS), J2.B9 (VBUS), U3.3 (INPUT)
- new net: J2.A5 (CC1), R5.1
- new net: J2.A6 (D+), J2.B6 (D+), R4.1
- new net: J2.A7 (D-), J2.B7 (D-), R3.1
- new net: J2.B5 (CC2), R6.1

Commit message: Fixes
- Changed to RP2350A
- Revised usb power
Parts:
- removed C1, C10, C2, C3, C4, C5, C6, C7, C8, C9: 100n, symbol Device:C_Small
- removed C11, C12, C13: 4.7u, symbol Device:C_Small
- removed C16: 10u, symbol Device:C_Small
- removed J1: SM03B-SRSS-TBLFSN, CONN_SM03B-SRSS-TB_JST, symbol Symbols:SM03B-SRSS-TBLFSN
- removed J3: Conn_01x13_Pin, symbol Connector:Conn_01x13_Pin
- removed J4: Conn_2Rows-51Pins, symbol Connector_Generic:Conn_2Rows-51Pins
- removed R1: R, symbol Device:R
- removed U1: RP2350B, Package_DFN_QFN:QFN-80-1EP_10x10mm_P0.4mm_EP3.4x3.4mm, symbol MCU_RaspberryPi:RP2350B
- removed U3: NCP1117ST33T3G, SOT223-3_ONS, symbol Symbols:NCP1117ST33T3G
- added C19, C20, C24, C32: 4.7u, symbol Device:C_Small
- added C21: 47u, symbol Device:C_Small
- added C22, C23, C25, C26, C27, C28, C29, C30, C31: 100n, symbol Device:C_Small
- added CR1: USBLC6-2SC6, SOT23-6L_STM, symbol Symbols:USBLC6-2SC6
- added D1: PMEG6010ELR, Diode_SMD:Nexperia_CFP3_SOD-123W, symbol Diode:PMEG6010ELR
- added J1: Conn_01x03_Pin, symbol Connector:Conn_01x03_Pin
- added J3: Conn_02x20_Top_Bottom, symbol Connector_Generic:Conn_02x20_Top_Bottom
- added L2: AOTA-B201610S3R3-101-T, IND_AOTA-B201610S_2p0x1p6x1p0_ABR, symbol Symbols:AOTA-B201610S3R3-101-T
- added R10: 5.6k, symbol Device:R
- added R11: 10k, symbol Device:R
- added R12, R13: 100k, symbol Device:R
- added R7: 1, symbol Device:R
- added R8: 200, symbol Device:R
- added R9: 33, symbol Device:R
- added U1: RP2350A, Package_DFN_QFN:QFN-60-1EP_7x7mm_P0.4mm_EP3.4x3.4mm, symbol MCU_RaspberryPi:RP2350A
- added U3: RT6150B-33GQW, 10-WFDFN-EP_RIT, symbol Symbols:RT6150B-33GQW
- C17: value 10u -> 4.7u
- L1: value 3.3u -> 2.2u
Connections:
- net +1V1: now also C20.2, C22.1, C23.1, C24.1, L2.1, U1.23 (DVDD), U1.39 (DVDD), U1.50 (VREG_FB), U1.6 (DVDD); no longer L1.1
- net GND: now also C19.1, C20.1, C21.2, C22.2, C23.2, C24.2, C25.1, C26.1, C27.1, C28.1, C29.1, C30.1, C31.1, C32.1, CR1.2, J1.2 (Pin_2), J3.13 (Pin_13), J3.18 (Pin_18), J3.23 (Pin_23), J3.28 (Pin_28), J3.3 (Pin_3), J3.33 (Pin_33), J3.38 (Pin_38), J3.8 (Pin_8), R11.2, R12.1, U1.47 (VREG_PGND), U1.61 (GND), U3.11 (GND), U3.3 (GND), U3.9 (GND)
- net QSPI_SCLK: now also U1.56 (QSPI_SCLK)
- net QSPI_SD0: now also U1.57 (QSPI_SD0)
- net QSPI_SD1: now also U1.59 (QSPI_SD1)
- net QSPI_SD2: now also U1.58 (QSPI_SD2)
- net QSPI_SD3: now also U1.55 (QSPI_SD3)
- net QSPI_SS: now also U1.60 (~{QSPI_SS})
- net at R2.2: now also U1.22 (XOUT)
- net VBUS: now reaches J2.A4 (VBUS), J2.A9 (VBUS), J2.B4 (VBUS), J2.B9 (VBUS)
- net VBUS: now also CR1.5, D1.2 (A), J3.21 (Pin_21), R10.1; no longer C17.1
- net at J2.A6 (D+), J2.B6 (D+): now also CR1.3; no longer R4.1
- net at J2.A7 (D-), J2.B7 (D-): now also CR1.1; no longer R3.1
- net at C15.1, X1.1: now also U1.21 (XIN)
- net at L1.2: now also U3.2 (LX2)
- net at R3.2: now also U1.51 (USB_DM)
- net at R4.2: now also U1.52 (USB_DP)
- net +3V3 renamed +3.3V
- net +3.3V: now also C25.2, C26.2, C27.2, C28.2, C29.2, C30.2, C31.2, C32.2, J3.25 (Pin_25), R8.1, R9.2, U1.1 (IOVDD), U1.11 (IOVDD), U1.20 (IOVDD), U1.30 (IOVDD), U1.38 (IOVDD), U1.45 (IOVDD), U1.49 (VREG_VIN), U1.53 (USB_OTP_VDD), U1.54 (QSPI_IOVDD), U3.1 (VOUT), U3.10 (FB)
- new net: CR1.6, R3.1
- new net: C19.2, R7.2, U1.44 (ADC_AVDD)
- new net: L1.1, U3.4 (LX1)
- new net: CR1.4, R4.1
- new net: C17.1, R9.1, U1.46 (VREG_AVDD)
- new net: J1.1 (Pin_1), U1.24 (SWCLK)
- new net: J1.3 (Pin_3), U1.25 (SWDIO)
- new net: L2.2, U1.48 (VREG_LX)
- new net 3V3_EN: J3.24 (Pin_24), R13.2, U3.6 (EN)
- new net ADC_VREF: J3.26 (Pin_26), R7.1, R8.2
- new net GPIO0: J3.1 (Pin_1), U1.2 (GPIO0)
- new net GPIO1: J3.2 (Pin_2), U1.3 (GPIO1)
- new net GPIO10: J3.14 (Pin_14), U1.14 (GPIO10)
- new net GPIO11: J3.15 (Pin_15), U1.15 (GPIO11)
- new net GPIO12: J3.16 (Pin_16), U1.16 (GPIO12)
- new net GPIO13: J3.17 (Pin_17), U1.17 (GPIO13)
- new net GPIO14: J3.19 (Pin_19), U1.18 (GPIO14)
- new net GPIO15: J3.20 (Pin_20), U1.19 (GPIO15)
- new net GPIO16: J3.40 (Pin_40), U1.27 (GPIO16)
- new net GPIO17: J3.39 (Pin_39), U1.28 (GPIO17)
- new net GPIO18: J3.37 (Pin_37), U1.29 (GPIO18)
- new net GPIO19: J3.36 (Pin_36), U1.31 (GPIO19)
- new net GPIO2: J3.4 (Pin_4), U1.4 (GPIO2)
- new net GPIO20: J3.35 (Pin_35), U1.32 (GPIO20)
- new net GPIO21: J3.34 (Pin_34), U1.33 (GPIO21)
- new net GPIO22: J3.32 (Pin_32), U1.34 (GPIO22)
- new net GPIO23: R12.2, U1.35 (GPIO23), U3.7 (PS)
- new net GPIO24: R10.2, R11.1, U1.36 (GPIO24)
- new net GPIO25: U1.37 (GPIO25)
- new net GPIO26/ADC0: J3.30 (Pin_30), U1.40 (GPIO26/ADC0)
- new net GPIO27/ADC1: J3.29 (Pin_29), U1.41 (GPIO27/ADC1)
- new net GPIO28/ADC2: J3.27 (Pin_27), U1.42 (GPIO28/ADC2)
- new net GPIO29/ADC3: U1.43 (GPIO29/ADC3)
- new net GPIO3: J3.5 (Pin_5), U1.5 (GPIO3)
- new net GPIO4: J3.6 (Pin_6), U1.7 (GPIO4)
- new net GPIO5: J3.7 (Pin_7), U1.8 (GPIO5)
- new net GPIO6: J3.9 (Pin_9), U1.9 (GPIO6)
- new net GPIO7: J3.10 (Pin_10), U1.10 (GPIO7)
- new net GPIO8: J3.11 (Pin_11), U1.12 (GPIO8)
- new net GPIO9: J3.12 (Pin_12), U1.13 (GPIO9)
- new net RUN: J3.31 (Pin_31), U1.26 (RUN)
- new net VSYS: C21.1, D1.1 (K), J3.22 (Pin_22), R13.1, U3.5 (VIN), U3.8 (VINA)
Other:
- moved on the sheet: R2

Commit message: Test
Parts:
- C14, C15, C17, C18, C19, C20, C21, C22, C23, C24, C25, C26, C27, C28, C29, C30, C31, C32: footprint (none) -> Capacitor_SMD:CP_Elec_5x5.9
- J1: footprint (none) -> Connector_PinHeader_2.00mm:PinHeader_1x03_P2.00mm_Horizontal
- J2: footprint (none) -> Connector_USB:USB_C_Receptacle_GCT_USB4110
- J3: footprint (none) -> Connector_PinHeader_2.00mm:PinHeader_2x20_P2.00mm_Vertical
- L1, R2: footprint (none) -> Inductor_SMD:L_0201_0603Metric_Pad0.64x0.40mm_HandSolder
- R10, R11, R12, R13, R3, R4, R5, R6, R7, R8, R9: footprint (none) -> Resistor_SMD:R_1020_2550Metric_Pad1.33x5.20mm_HandSolder

Commit message: Fixes
Parts:
- added C33: 1n, Capacitor_SMD:CP_Elec_5x5.9, symbol MCU_Project:C_Small
- added D2: LED, symbol Device:LED
- added Q1: DMG1012T, Package_TO_SOT_SMD:SOT-523, symbol Transistor_FET:DMG1012T
- added R14: 470, Resistor_SMD:R_1020_2550Metric_Pad1.33x5.20mm_HandSolder, symbol MCU_Project:R
- added R15, R16, R17: 100k, Resistor_SMD:R_1020_2550Metric_Pad1.33x5.20mm_HandSolder, symbol MCU_Project:R
- C14, C15, C17, C18, C19, C20, C21, C22, C23, C24, C25, C26, C27, C28, C29, C30, C31, C32: symbol Device:C_Small -> MCU_Project:C_Small
- CR1: footprint SOT23-6L_STM -> MCU_Footprints:SOT23-6L_STM; symbol Symbols:USBLC6-2SC6 -> MCU_Project:USBLC6-2SC6
- D1: symbol Diode:PMEG6010ELR -> MCU_Project:PMEG6010ELR
- J1: symbol Connector:Conn_01x03_Pin -> MCU_Project:Conn_01x03_Pin
- J2: symbol Connector:USB_C_Receptacle_USB2.0_14P -> MCU_Project:USB_C_Receptacle_USB2.0_14P
- J3: symbol Connector_Generic:Conn_02x20_Top_Bottom -> MCU_Project:Conn_02x20_Top_Bottom
- L1: symbol Device:L -> MCU_Project:L
- L2: footprint IND_AOTA-B201610S_2p0x1p6x1p0_ABR -> MCU_Footprints:IND_AOTA-B201610S_2p0x1p6x1p0_ABR; symbol Symbols:AOTA-B201610S3R3-101-T -> MCU_Project:AOTA-B201610S3R3-101-T
- R10, R11, R12, R13, R2, R3, R4, R5, R6, R7, R8, R9: symbol Device:R -> MCU_Project:R
- U1: symbol MCU_RaspberryPi:RP2350A -> MCU_Project:RP2350A
- U2: footprint SOIC_128JVSIQ_WIN -> MCU_Footprints:SOIC_128JVSIQ_WIN; symbol Symbols:W25Q128JVSIQ -> MCU_Project:W25Q128JVSIQ
- U3: footprint 10-WFDFN-EP_RIT -> MCU_Footprints:10-WFDFN-EP_RIT; symbol Symbols:RT6150B-33GQW -> MCU_Project:RT6150B-33GQW
- X1: footprint ABM8-272-T3_ABR -> MCU_Footprints:ABM8-272-T3_ABR; symbol 2026-10-15_16-24-31:ABM8-272-T3 -> MCU_Project:ABM8-272-T3
Connections:
- net +3.3V: now also Q1.1 (G)
- net GND: now also C33.1, D2.1 (K), R15.2, R16.1
- net GPIO25: now also R14.1
- net GPIO29/ADC3: now also Q1.3 (D), R15.1
- net VSYS: now also R17.1
- new net: C33.2, Q1.2 (S), R16.2, R17.2
- new net: D2.2 (A), R14.2
